File: kicad/paste_dispenser/paste_dispenser.sch (KiCad schematic (older format))
At the start: 24 parts, among them J1 ISP, J2 EXT, J3 STEPPER, J4 OLED, Q1 SSM3J328R_LF, SW1 SW_PB, SW2 SW_PB, SW3 SW_PB, SW4 SW_PB, U1 ATmega328P-AU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

Commit message: add header
Parts:
- J2: Manufacturer Molex -> TE; Manufacturer Part No 70553-0005 -> 5-102203-3; Note Mates with Molex 50-57-9406 -> Mates with Dupont connectors; Source 1 Part No 538-70553-0005 -> 571-5-102203-3
Changed lines of the file:
@@
 F 2 "Connector_PinHeader_2.54mm:PinHeader_1x06_P2.54mm_Vertical" H 5700 4400 50  0001 C CNN
 F 3 "~" H 5700 4400 50  0001 C CNN
-F 4 "Molex" H 5700 4400 50  0001 C CNN "Manufacturer"
-F 5 "70553-0005" H 5700 4400 50  0001 C CNN "Manufacturer Part No"
+F 4 "TE" H 5700 4400 50  0001 C CNN "Manufacturer"
+F 5 "5-102203-3" H 5700 4400 50  0001 C CNN "Manufacturer Part No"
 F 6 "mouser.com" H 5700 4400 50  0001 C CNN "Source 1"
-F 7 "538-70553-0005" H 5700 4400 50  0001 C CNN "Source 1 Part No"
-F 8 "Mates with Molex 50-57-9406" H 5700 4400 50  0001 C CNN "Note"
+F 7 "571-5-102203-3" H 5700 4400 50  0001 C CNN "Source 1 Part No"
+F 8 "Mates with Dupont connectors" H 5700 4400 50  0001 C CNN "Note"
 	1    5700 4400
 	1    0    0    -1
